File: kicad/sweek_rdmxchoc/sweek_rdmxchoc.kicad_sch (KiCad schematic)
At the start: 60 parts, among them J1 Conn_01x04_Socket, J2 OLED_128x32, SW1 RotaryEncoder_Switch, U1 RP2040_Zero

Commit message: Update sweek kicad files for v1.0.1
Update sweek kicad files for v1.0.1
Parts:
- D1, D10, D11, D12, D13, D14, D15, D16, D17, D18, D2, D3, D4, D5, D6, D7, D8, D9: footprint ScottoKeebs_Components:Diode_DO-35 -> Redragon:Diode_DO-35_SOD-123
- JP1: footprint Jumper:SolderJumper-2_P1.3mm_Open_TrianglePad1.0x1.5mm -> Jumper:SolderJumper-2_P1.3mm_Open_TrianglePad1.0x1.5mm_custom
- JP10, JP11, JP2, JP3, JP4, JP5, JP6, JP7, JP9: footprint Jumper:SolderJumper-2_P1.3mm_Open_RoundedPad1.0x1.5mm -> Jumper:SolderJumper-2_P1.3mm_Open_RoundedPad1.0x1.5mm_custom
- JP8: footprint Jumper:SolderJumper-2_P1.3mm_Bridged_RoundedPad1.0x1.5mm -> Jumper:SolderJumper-2_P1.3mm_Bridged_RoundedPad1.0x1.5mm_custom
- R1, R2, R3, R4, R5: footprint Resistor_SMD:R_1206_3216Metric_Pad1.30x1.75mm_HandSolder -> Resistor_SMD:R_1206_3216Metric_Pad1.30x1.75mm_custom
Changed lines of the file:
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@@
 			)
 		)
-		(property "Footprint" "ScottoKeebs_Components:Diode_DO-35"
+		(property "Footprint" "Redragon:Diode_DO-35_SOD-123"
 			(at 83.82 86.36 0)
 			(effects
@@
 			)
 		)
-		(property "Footprint" "ScottoKeebs_Components:Diode_DO-35"
+		(property "Footprint" "Redragon:Diode_DO-35_SOD-123"
 			(at 71.12 66.04 0)
 			(effects
@@
 			)
 		)
-		(property "Footprint" "Resistor_SMD:R_1206_3216Metric_Pad1.30x1.75mm_HandSolder"
+		(property "Footprint" "Resistor_SMD:R_1206_3216Metric_Pad1.30x1.75mm_custom"
 			(at 215.9 105.918 0)
 			(effects
@@
 			)
 		)
-		(property "Footprint" "ScottoKeebs_Components:Diode_DO-35"
+		(property "Footprint" "Redragon:Diode_DO-35_SOD-123"
 			(at 109.22 86.36 0)
 			(effects
@@
 			)
 		)
-		(property "Footprint" "Resistor_SMD:R_1206_3216Metric_Pad1.30x1.75mm_HandSolder"
+		(property "Footprint" "Resistor_SMD:R_1206_3216Metric_Pad1.30x1.75mm_custom"
 			(at 156.21 74.168 0)
 			(effects
@@
 			)
 		)
-		(property "Footprint" "Jumper:SolderJumper-2_P1.3mm_Open_RoundedPad1.0x1.5mm"
+		(property "Footprint" "Jumper:SolderJumper-2_P1.3mm_Open_RoundedPad1.0x1.5mm_custom"
 			(at 161.29 100.33 0)
 			(effects
@@
 			)
 		)
-		(property "Footprint" "ScottoKeebs_Components:Diode_DO-35"
+		(property "Footprint" "Redragon:Diode_DO-35_SOD-123"
 			(at 109.22 66.04 0)
 			(effects
@@
 			)
 		)
-		(property "Footprint" "Jumper:SolderJumper-2_P1.3mm_Open_RoundedPad1.0x1.5mm"
+		(property "Footprint" "Jumper:SolderJumper-2_P1.3mm_Open_RoundedPad1.0x1.5mm_custom"
 			(at 234.95 88.9 0)
 			(effects
@@
 			)
 		)
-		(property "Footprint" "ScottoKeebs_Components:Diode_DO-35"
+		(property "Footprint" "Redragon:Diode_DO-35_SOD-123"
 			(at 96.52 45.72 0)
 			(effects
@@
 			)
 		)
-		(property "Footprint" "Jumper:SolderJumper-2_P1.3mm_Open_RoundedPad1.0x1.5mm"
+		(property "Footprint" "Jumper:SolderJumper-2_P1.3mm_Open_RoundedPad1.0x1.5mm_custom"
 			(at 219.71 119.38 0)
 			(effects
@@
 			)
 		)
-		(property "Footprint" "Jumper:SolderJumper-2_P1.3mm_Open_RoundedPad1.0x1.5mm"
+		(property "Footprint" "Jumper:SolderJumper-2_P1.3mm_Open_RoundedPad1.0x1.5mm_custom"
 			(at 237.49 88.9 0)
 			(effects
@@
 			)
 		)
-		(property "Footprint" "Resistor_SMD:R_1206_3216Metric_Pad1.30x1.75mm_HandSolder"
+		(property "Footprint" "Resistor_SMD:R_1206_3216Metric_Pad1.30x1.75mm_custom"
 			(at 156.21 76.708 0)
 			(effects
@@
 			)
 		)
-		(property "Footprint" "Jumper:SolderJumper-2_P1.3mm_Open_RoundedPad1.0x1.5mm"
+		(property "Footprint" "Jumper:SolderJumper-2_P1.3mm_Open_RoundedPad1.0x1.5mm_custom"
 			(at 219.71 121.92 0)
 			(effects
@@
 			)
 		)
-		(property "Footprint" "ScottoKeebs_Components:Diode_DO-35"
+		(property "Footprint" "Redragon:Diode_DO-35_SOD-123"
 			(at 83.82 66.04 0)
 			(effects
@@
 			)
 		)
-		(property "Footprint" "ScottoKeebs_Components:Diode_DO-35"
+		(property "Footprint" "Redragon:Diode_DO-35_SOD-123"
 			(at 118.11 109.22 0)
 			(effects
@@
 			)
 		)
-		(property "Footprint" "ScottoKeebs_Components:Diode_DO-35"
+		(property "Footprint" "Redragon:Diode_DO-35_SOD-123"
 			(at 109.22 45.72 0)
 			(effects
@@
 			)
 		)
-		(property "Footprint" "ScottoKeebs_Components:Diode_DO-35"
+		(property "Footprint" "Redragon:Diode_DO-35_SOD-123"
 			(at 71.12 86.36 0)
 			(effects
@@
 			)
 		)
-		(property "Footprint" "ScottoKeebs_Components:Diode_DO-35"
+		(property "Footprint" "Redragon:Diode_DO-35_SOD-123"
 			(at 71.12 45.72 0)
 			(effects
@@
 			)
 		)
-		(property "Footprint" "Jumper:SolderJumper-2_P1.3mm_Bridged_RoundedPad1.0x1.5mm"
+		(property "Footprint" "Jumper:SolderJumper-2_P1.3mm_Bridged_RoundedPad1.0x1.5mm_custom"
 			(at 219.71 124.46 0)
 			(effects
@@
 			)
 		)
-		(property "Footprint" "ScottoKeebs_Components:Diode_DO-35"
+		(property "Footprint" "Redragon:Diode_DO-35_SOD-123"
 			(at 105.41 109.22 0)
 			(effects
@@
 			)
 		)
-		(property "Footprint" "ScottoKeebs_Components:Diode_DO-35"
+		(property "Footprint" "Redragon:Diode_DO-35_SOD-123"
 			(at 96.52 66.04 0)
 			(effects
@@
 			)
 		)
-		(property "Footprint" "ScottoKeebs_Components:Diode_DO-35"
+		(property "Footprint" "Redragon:Diode_DO-35_SOD-123"
 			(at 83.82 45.72 0)
 			(effects
@@
 			)
 		)
-		(property "Footprint" "ScottoKeebs_Components:Diode_DO-35"
+		(property "Footprint" "Redragon:Diode_DO-35_SOD-123"
 			(at 96.52 86.36 0)
 			(effects
@@
 			)
 		)
-		(property "Footprint" "ScottoKeebs_Components:Diode_DO-35"
+		(property "Footprint" "Redragon:Diode_DO-35_SOD-123"
 			(at 58.42 86.36 0)
 			(effects
@@
 			)
 		)
-		(property "Footprint" "Jumper:SolderJumper-2_P1.3mm_Open_RoundedPad1.0x1.5mm"
+		(property "Footprint" "Jumper:SolderJumper-2_P1.3mm_Open_RoundedPad1.0x1.5mm_custom"
 			(at 161.29 105.41 0)
 			(effects
@@
 			)
 		)
-		(property "Footprint" "ScottoKeebs_Components:Diode_DO-35"
+		(property "Footprint" "Redragon:Diode_DO-35_SOD-123"
 			(at 58.42 45.72 0)
 			(effects
@@
 			)
 		)
-		(property "Footprint" "Jumper:SolderJumper-2_P1.3mm_Open_TrianglePad1.0x1.5mm"
+		(property "Footprint" "Jumper:SolderJumper-2_P1.3mm_Open_TrianglePad1.0x1.5mm_custom"
 			(at 248.92 59.69 0)
 			(effects
@@
 			)
 		)
-		(property "Footprint" "Resistor_SMD:R_1206_3216Metric_Pad1.30x1.75mm_HandSolder"
+		(property "Footprint" "Resistor_SMD:R_1206_3216Metric_Pad1.30x1.75mm_custom"
 			(at 156.21 69.088 0)
 			(effects
@@
 			)
 		)
-		(property "Footprint" "ScottoKeebs_Components:Diode_DO-35"
+		(property "Footprint" "Redragon:Diode_DO-35_SOD-123"
 			(at 92.71 109.22 0)
 			(effects
@@
 			)
 		)
-		(property "Footprint" "Jumper:SolderJumper-2_P1.3mm_Open_RoundedPad1.0x1.5mm"
+		(property "Footprint" "Jumper:SolderJumper-2_P1.3mm_Open_RoundedPad1.0x1.5mm_custom"
 			(at 215.9 99.06 0)
 			(effects
@@
 			)
 		)
-		(property "Footprint" "Jumper:SolderJumper-2_P1.3mm_Open_RoundedPad1.0x1.5mm"
+		(property "Footprint" "Jumper:SolderJumper-2_P1.3mm_Open_RoundedPad1.0x1.5mm_custom"
 			(at 215.9 101.6 0)
 			(effects
@@
 			)
 		)
-		(property "Footprint" "Jumper:SolderJumper-2_P1.3mm_Open_RoundedPad1.0x1.5mm"
+		(property "Footprint" "Jumper:SolderJumper-2_P1.3mm_Open_RoundedPad1.0x1.5mm_custom"
 			(at 215.9 106.68 0)
 			(effects
@@
 			)
 		)
-		(property "Footprint" "Resistor_SMD:R_1206_3216Metric_Pad1.30x1.75mm_HandSolder"
+		(property "Footprint" "Resistor_SMD:R_1206_3216Metric_Pad1.30x1.75mm_custom"
 			(at 156.21 71.628 0)
 			(effects
@@
 			)
 		)
-		(property "Footprint" "ScottoKeebs_Components:Diode_DO-35"
+		(property "Footprint" "Redragon:Diode_DO-35_SOD-123"
 			(at 58.42 66.04 0)
 			(effects
